File: FMC_Extension/0001/Design/FMC_Fanout.sch (KiCad schematic (older format))
At the start: 2 parts, among them J1 ASP-134488-01_MALE, J2 Conn_Coaxial

Commit message: Test_Cadlab_dbaudin
Connections:
- wire segments 0 -> 5
Changed lines of the file:
@@
 Text Notes 1625 7175 0    50   ~ 0
 SMA\n
+Wire Wire Line
+	1500 5825 1200 5825
+Wire Wire Line
+	1200 5825 1200 6375
+Wire Wire Line
+	1200 6375 2925 6375
+Wire Wire Line
+	2925 5825 2925 6375
+Connection ~ 2925 6375
+Wire Wire Line
+	2925 6375 2925 6450
 $EndSCHEMATC

Commit message: Suppression jonction
Connections:
- wire segments 5 -> 4
Changed lines of the file:
@@
 Wire Wire Line
 	2925 5825 2925 6375
-Connection ~ 2925 6375
-Wire Wire Line
-	2925 6375 2925 6450
 $EndSCHEMATC
